File: pcb/nunchuck_mod.brd (EAGLE design)
At the start: 100 x 80 mm, 23 parts, among them J2 USB Micro, J3 Wii Nunchuck, J4 ICSP, U1 MCP73831, U2 ATTINY4313-SU

Commit message: Completed PCB design
Had to replace RGB led with 3 individual LEDs and completed PCB design
Parts:
- removed D1: (no value), SparkFun-LED:LED-TRICOLOR-5050
- removed JP1: JUMPER-SMT_2_NC_PASTE_SILK, SparkFun-Jumpers:SMT-JUMPER_2_NC_PASTE_SILK
- added C3: 1.0uF, SparkFun-Capacitors:0603
- added C4, C5: 10uF, SparkFun-Capacitors:0603-POLAR
- added D2: RED, SparkFun-LED:LED-0603
- added D3: GREEN, SparkFun-LED:LED-0603
- added D4: BLUE, SparkFun-LED:LED-0603
- added J5: Power Switch, SparkFun-Connectors:1X02
- added U3: 3.3V/150mA, SparkFun-IC-Power:SOT23-5
- R7, R8: value 68OHM-0603-1/10W-1% -> 68OHM
- moved R12 180.5 mm to (1.88, 15.3), turned to 90 degrees
- moved R11 176.9 mm to (1.89, 15.2), flipped to the bottom, turned to 270 degrees
- moved J4 168.2 mm to (17.8, 13.7), flipped to the bottom, turned to 270 degrees
- moved R8 158.6 mm to (25.3, 19.1), turned to 270 degrees
- moved R7 152.8 mm to (22.7, 19.0), turned to 270 degrees
- moved R10 150.3 mm to (7.52, 9.84), turned to 180 degrees
- moved R9 144.9 mm to (7.56, 7.69), turned to 180 degrees
- moved J2 129.8 mm to (30.3, 21.9), turned to 180 degrees
- moved C2 122.3 mm to (29.2, 19.9), turned to 180 degrees
- moved J3 115.1 mm to (1.66, 1.90), turned to 90 degrees
- moved C1 105.6 mm to (3.48, 21.5), turned to 270 degrees
- moved R6 103.3 mm to (16.0, 21.1), flipped to the bottom, turned to 270 degrees
- moved R5 101.5 mm to (16.0, 22.8), turned to 90 degrees
- moved R1 85.3 mm to (10.4, 18.4), turned to 90 degrees
- moved R4 75.1 mm to (20.2, 19.6), flipped to the bottom, turned to 270 degrees
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Connections:
- removed net N$14: JP1.1, U$1.16, U2.9
- removed net N$9: J3.1
- removed net VIN: C2.2, R5.2, U1.4
- new net N$8: U$1.15, U$1.16
- net 3.3V: now also C3.1, C4.+, U3.5
- net GND: now also C3.2, C4.-, C5.-, D3.C, D4.C, J1.2, J3.1, U3.2; no longer D1.4, D1.6, J1.1
- net N$10: now also D2.A; no longer D1.2
- net N$13: now also J5.2, U3.3; no longer JP1.2, U$1.15, U2.8
- net N$15: now also R11.2; no longer R12.1
- net N$16: now also D2.C; no longer D1.5
- net N$22: now also R12.1; no longer R11.2
- net N$3: now also R2.2; no longer R2.1
- net N$4: now also D4.A, R2.1; no longer D1.3, R2.2
- net N$5: now also D3.A; no longer D1.1
- net V_BATT: now also C5.+, J1.1, J5.1, U3.1; no longer J1.2
- net V_USB: now also C2.2, R5.2, U1.4
Routing:
- net GND: track 0.00 -> 99.6 mm, vias 0 -> 3
- net 3.3V: track 0.00 -> 55.6 mm, vias 0 -> 3
- net N$22: track 0.00 -> 53.4 mm, vias 0 -> 3
- net N$15: track 0.00 -> 41.5 mm, vias 0 -> 3
- net N$18: track 0.00 -> 29.5 mm, vias 0 -> 2
- net N$12: track 0.00 -> 23.8 mm, vias 0 -> 2
- net V_USB: track 0.00 -> 19.7 mm, vias 0 -> 1
- net N$21: track 0.00 -> 19.4 mm, vias 0 -> 1
- net V_BATT: track 0.00 -> 18.1 mm, vias 0 -> 2
- net N$13: track 0.00 -> 7.63 mm
- net N$6: track 0.00 -> 6.32 mm, vias 0 -> 1
- net N$23: track 0.00 -> 5.92 mm, vias 0 -> 1
- net N$7: track 0.00 -> 5.10 mm, vias 0 -> 1
- net N$16: track 0.00 -> 4.63 mm, vias 0 -> 1
- net N$5: track 0.00 -> 3.35 mm, vias 0 -> 1
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Other:
- board size 100 x 80 mm -> 32 x 27 mm
