File: pcb/nunchuck_mod.sch (EAGLE design)
At the start: 23 parts, among them J2 USB Micro, J3 Wii Nunchuck, J4 ICSP, U1 MCP73831, U2 ATTINY4313-SU

Commit message: Completed PCB design
Had to replace RGB led with 3 individual LEDs and completed PCB design
Parts:
- removed D1: (no value), SparkFun-LED:LED-RGBNO_IC
- removed JP1: JUMPER-SMT_2_NC_PASTE_SILK, SparkFun-Jumpers:JUMPER-SMT_2_NC_PASTE_SILK
- added C3: 1.0uF, SparkFun-Capacitors:1.0UF-0603-16V-10%
- added C4, C5: 10uF, SparkFun-Capacitors:10UF-POLAR-0603-6.3V-20%(TANT)
- added D2: RED, SparkFun-LED:LED-RED0603
- added D3: GREEN, SparkFun-LED:LED-GREEN0603
- added D4: BLUE, SparkFun-LED:LED-BLUE0603
- added J5: Power Switch, SparkFun-Connectors:CONN_02
- added U3: 3.3V/150mA, SparkFun-IC-Power:V_REG_MIC52053.3V
- R7, R8: value 68OHM-0603-1/10W-1% -> 68OHM
Connections:
- removed net N$14: JP1.1, U$1.UARTCTS, U2.PD5
- removed net N$9: J3.1
- removed net VIN: C2.2, R5.2, U1.VIN
- new net N$8: U$1.UARTCTS, U$1.UARTRTS
- net 3.3V: now also C3.1, C4.+, U3.OUT
- net GND: now also C3.2, C4.-, C5.-, D3.C, D4.C, J1.+, J3.1, U3.GND; no longer D1.BLU-C, D1.GRN-C, J1.-
- net N$10: now also D2.A; no longer D1.RED-A
- net N$13: now also J5.2, U3.EN; no longer JP1.2, U$1.UARTRTS, U2.PD4
- net N$15: now also R11.2; no longer R12.1
- net N$16: now also D2.C; no longer D1.RED-C
- net N$22: now also R12.1; no longer R11.2
- net N$3: now also R2.2; no longer R2.1
- net N$4: now also D4.A, R2.1; no longer D1.BLU-A, R2.2
- net N$5: now also D3.A; no longer D1.GRN-A
- net V_BATT: now also C5.+, J1.-, J5.1, U3.IN; no longer J1.+
- net V_USB: now also C2.2, R5.2, U1.VIN
Other:
- moved on the sheet: C1, C2, J1, J3, R11, R12, R2, R5, R6, U1
